Commit message: Added mimic joint, colors.

File: robots/schunkPG70_description.URDF (robot description, URDF)
Before this commit: robot schunkPG70_description, 3 links, 2 joints
Links:
- link gripper_a_frame: mass 0.014276 -> 0.020334; geometry collision mesh filename=package://schunkPG70_description/meshes/gripper_frame.STL; visual mesh filename=package://schunkPG70_description/meshes/gripper_frame.STL
- link gripper_b_frame: mass 0.014276 -> 0.0203342527020743; geometry collision mesh filename=package://schunkPG70_description/meshes/gripper_frame.STL; visual mesh filename=package://schunkPG70_description/meshes/gripper_frame.STL
- link tool_frame: mass 0.77467 -> 0.965844004259551
Joints:
- joint gripper_b: axis 1 0 0 -> -1 0 0; origin xyz=0.0985 0.0323 0.00025 rpy=0 0 -1.5708 -> xyz=0.0985 0.0323 0.00025 rpy=3.1416 0 1.5708

Commit message: Added tool changer.

File: robots/schunkPG70_description.URDF (robot description, URDF)
Before this commit: robot schunkPG70_description, 3 links, 2 joints
Links:
- removed link tool_frame
- added link tool_link, mass 1.08662283556797; collision mesh filename=package://schunkPG70_description/meshes/tool_link.STL; visual mesh filename=package://schunkPG70_description/meshes/tool_link.STL
- link gripper_a_frame: mass 0.020334 -> 0.0203342527020743
Joints:
- joint gripper_a: origin xyz=0.0985 -0.0323 -0.00025 rpy=0 0 -1.5708 -> xyz=0.122275 0.0322999 0.000250099999999993 rpy=-3.14159265358979 -9.0205620750794E-17 1.5707963267949; parent tool_frame -> tool_link
- joint gripper_b: origin xyz=0.0985 0.0323 0.00025 rpy=3.1416 0 1.5708 -> xyz=0.122275 -0.0323001 -0.00024990000000001 rpy=-5.17444897013869E-31 9.0205620750794E-17 -1.5707963267949; parent tool_frame -> tool_link
