Commit message: Fixed name and added launchfile tests.

File: robots/schunk_pg70_description.URDF (robot description, URDF)
Before this commit: robot schunkPG70_description, 3 links, 2 joints
Links:
- link gripper_a_frame: geometry collision mesh filename=package://schunk_pg70_description/meshes/gripper_frame.STL; visual mesh filename=package://schunk_pg70_description/meshes/gripper_frame.STL
- link gripper_b_frame: geometry collision mesh filename=package://schunk_pg70_description/meshes/gripper_frame.STL; visual mesh filename=package://schunk_pg70_description/meshes/gripper_frame.STL
- link tool_frame: geometry collision mesh filename=package://schunk_pg70_description/meshes/tool_frame.STL; visual mesh filename=package://schunk_pg70_description/meshes/tool_frame.STL
